File: kicad/RT1176.kicad_sch (KiCad schematic)
At the start: 0 parts

Commit message: switching to laptop
Changed lines of the file:
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@@
 	(paper "A4")
 	(sheet
-		(at 68.58 21.59)
-		(size 35.56 24.13)
+		(at 68.58 22.86)
+		(size 52.07 29.21)
 		(exclude_from_sim no)
 		(in_bom yes)
@@
 		)
 		(property "Sheetname" "RT1176_1"
-			(at 68.58 20.8784 0)
+			(at 68.58 22.1484 0)
 			(effects
 				(font
@@
 		)
 		(property "Sheetfile" "RT1176_1.kicad_sch"
-			(at 68.58 46.3046 0)
+			(at 68.58 52.6546 0)
 			(effects
 				(font
@@
 	)
 	(sheet
-		(at 68.58 105.41)
-		(size 49.53 34.29)
+		(at 68.58 96.52)
+		(size 52.07 34.29)
 		(exclude_from_sim no)
 		(in_bom yes)
@@
 		)
 		(property "Sheetname" "RT1176_3"
-			(at 68.58 104.6984 0)
+			(at 68.58 95.8084 0)
 			(effects
 				(font
@@
 		)
 		(property "Sheetfile" "RT1176_3.kicad_sch"
-			(at 68.58 140.2846 0)
+			(at 68.58 131.3946 0)
 			(effects
 				(font
@@
 	)
 	(sheet
-		(at 68.58 60.96)
-		(size 36.83 29.21)
+		(at 68.58 58.42)
+		(size 52.07 31.75)
 		(exclude_from_sim no)
 		(in_bom yes)
@@
 		)
 		(property "Sheetname" "RT1176_2"
-			(at 68.58 60.2484 0)
+			(at 68.58 57.7084 0)
 			(effects
 				(font
